File: 65-wkl-pcb.kicad_pcb (KiCad board)
At the start: 2 copper layers, 168 parts, among them J1 USB_C_Receptacle_USB2.0_16P, J2 Conn_01x04, J3 Conn_01x05, U1 XC6206PxxxMR, U2 SRV05-4, U3 RP2040, U4 W25Q128JVS, Y1 Crystal_GND24

Commit message: updating
Parts:
- added J4: Conn_01x04, Connector_JST:JST_PH_S4B-PH-K_1x04_P2.00mm_Horizontal, B.Cu at (181.0, 116.5)
- F1, J1, J2, R1, R2, U2: moved to F.Cu
- moved U2 102.2 mm to (122.7, 116.5), turned to 0 degrees
- moved F1 20.6 mm to (23.8, 161.1), turned to 0 degrees
- moved R2 13.9 mm to (36.0, 161.3), turned to 180 degrees
- moved J1 9.59 mm to (38.9, 154.8), turned to 180 degrees
- moved J2 9.56 mm to (34.9, 169.9), turned to 0 degrees
- moved R1 6.32 mm to (41.4, 161.3), turned to 0 degrees
Routing:
- net D+: track 0.00 -> 3.10 mm
- net Net-(J1-CC1): track 0.00 -> 2.79 mm
- net Net-(J1-CC2): track 0.00 -> 2.75 mm

Commit message: daughterboard
Parts:
- removed C1, C2: 1u, Capacitor_SMD:C_0402_1005Metric
- removed F1: Fuse_Small, Fuse:Fuse_1206_3216Metric
- removed J1: USB_C_Receptacle_USB2.0_16P, Connector_USB:USB_C_Receptacle_HRO_TYPE-C-31-M-12
- removed J2: Conn_01x04, Connector_JST:JST_PH_S4B-PH-K_1x04_P2.00mm_Horizontal
- removed R1, R2: 5.1k, Resistor_SMD:R_0402_1005Metric
- removed U1: XC6206PxxxMR, Package_TO_SOT_SMD:SOT-23-3
- removed U2: SRV05-4, PCM_marbastlib-various:SOT-23-6-routable
- moved RST1 1.12 mm to (110.3, 154.8)
- moved C10 0.22 mm to (137.3, 131.2)
Connections:
- R4 pad 1: Q_SEL -> Net-(R4-Pad1)
- R5 pad 2: Q_SEL -> Net-(R4-Pad1)
Routing:
- net D+: track 3.10 -> 0.00 mm
- net Net-(J1-CC1): track 2.79 -> 0.00 mm
- net Net-(J1-CC2): track 2.75 -> 0.00 mm
